File: Connectivity/RFswitch/rfswitch.kicad_pcb (KiCad board)
At the start: 2 copper layers, 23 parts, among them P1 BNC, P2 BNC, P3 BNC, P4 BNC, P5 BNC, P6 CONN_01X02, SW1 SW_PUSH, SW2 SW_PUSH, SW3 SW_PUSH, SW4 SW_PUSH, U1 LT1129CS8

Commit message: trx model sim matlab initial
Routing:
- net Net-(P5-Pad1): track 0.00 -> 224.8 mm
- net Net-(RL1-PadA2): track 20.5 -> 195.7 mm
- net Net-(P4-Pad1): track 0.00 -> 11.7 mm
Other:
- net class rf50ohm18u added: clearance 2, trace_width 1.83, via_dia 2, via_drill 1.83
- rule trace_min: 0.2 -> 0.1
Changed lines of the file:
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@@
     (thickness 1.6)
     (drawings 0)
-    (tracks 10)
+    (tracks 54)
     (zones 0)
     (modules 23)
@@
   )
   (setup
-    (last_trace_width 0.25)
+    (last_trace_width 1.83)
+    (user_trace_width 1.83)
     (trace_clearance 0.2)
     (zone_clearance 0.508)
     (zone_45_only no)
-    (trace_min 0.2)
+    (trace_min 0.1)
     (segment_width 0.2)
     (edge_width 0.15)
@@
     (via_min_size 0.4)
     (via_min_drill 0.3)
+    (user_via 2 1.83)
     (uvia_size 0.3)
     (uvia_drill 0.1)
@@
     (mod_text_size 1 1)
     (mod_text_width 0.15)
-    (pad_size 1.524 1.524)
-    (pad_drill 0.762)
+    (pad_size 2.99974 2.99974)
+    (pad_drill 1.19888)
     (pad_to_mask_clearance 0.2)
     (aux_axis_origin 0 0)
@@
     (add_net "Net-(U1-Pad6)")
   )
+  (net_class rf50ohm18u ""
+    (clearance 2)
+    (trace_width 1.83)
+    (via_dia 2)
+    (via_drill 1.83)
+    (uvia_dia 0.3)
+    (uvia_drill 0.1)
+  )
   (module Capacitors_SMD:c_elec_5x5.3 (layer F.Cu)
     (at 185.166 97.9424)
@@
   (segment (start 124.22886 73.7108) (end 130.6068 73.7108) (width 0.25) (layer F.Cu) (net 8))
   (segment (start 130.6068 73.7108) (end 133.9088 70.4088) (width 0.25) (layer F.Cu) (net 8))
-  (segment (start 160.8328 73.2028) (end 160.8328 86.7156) (width 0.25) (layer F.Cu) (net 17))
-  (segment (start 160.8328 86.7156) (end 158.6992 88.8492) (width 0.25) (layer F.Cu) (net 17))
-  (segment (start 158.0388 70.4088) (end 160.8328 73.2028) (width 0.25) (layer F.Cu) (net 17))
+  (segment (start 124.94006 130.7592) (end 131.2164 130.7592) (width 1.83) (layer F.Cu) (net 10))
+  (segment (start 131.2164 130.7592) (end 135.0772 126.8984) (width 1.83) (layer F.Cu) (net 10))
+  (segment (start 173.408599 87.976797) (end 173.408599 89.390801) (width 1.83) (layer F.Cu) (net 11))
+  (segment (start 139.839936 78.0288) (end 148.045465 86.234329) (width 1.83) (layer F.Cu) (net 11))
+  (segment (start 173.730598 89.7128) (end 193.612828 89.7128) (width 1.83) (layer F.Cu) (net 11))
+  (segment (start 193.612828 89.7128) (end 200.724828 96.8248) (width 1.83) (layer F.Cu) (net 11))
+  (segment (start 137.7188 78.0288) (end 139.839936 78.0288) (width 1.83) (layer F.Cu) (net 11))
+  (segment (start 148.045465 86.234329) (end 171.666131 86.234329) (width 1.83) (layer F.Cu) (net 11))
+  (segment (start 171.666131 86.234329) (end 173.408599 87.976797) (width 1.83) (layer F.Cu) (net 11))
+  (segment (start 173.408599 89.390801) (end 173.730598 89.7128) (width 1.83) (layer F.Cu) (net 11))
+  (segment (start 200.724828 96.8248) (end 201.85634 96.8248) (width 1.83) (layer F.Cu) (net 11))
+  (segment (start 165.862 102.9208) (end 165.862 101.793798) (width 1.83) (layer F.Cu) (net 11))
+  (segment (start 165.862 101.793798) (end 168.884399 98.771399) (width 1.83) (layer F.Cu) (net 11))
+  (segment (start 168.884399 98.771399) (end 174.468401 98.771399) (width 1.83) (layer F.Cu) (net 11))
+  (segment (start 174.468401 98.771399) (end 175.554503 99.857501) (width 1.83) (layer F.Cu) (net 11))
+  (segment (start 175.554503 99.857501) (end 198.823639 99.857501) (width 1.83) (layer F.Cu) (net 11))
+  (segment (start 198.823639 99.857501) (end 201.056241 97.624899) (width 1.83) (layer F.Cu) (net 11))
+  (segment (start 201.056241 97.624899) (end 201.85634 96.8248) (width 1.83) (layer F.Cu) (net 11))
+  (segment (start 152.9588 102.9208) (end 165.862 102.9208) (width 1.83) (layer F.Cu) (net 11))
+  (segment (start 141.352269 114.527331) (end 152.9588 102.9208) (width 1.83) (layer F.Cu) (net 11))
+  (segment (start 137.8712 116.0272) (end 139.371069 114.527331) (width 1.83) (layer F.Cu) (net 11))
+  (segment (start 139.371069 114.527331) (end 141.352269 114.527331) (width 1.83) (layer F.Cu) (net 11))
+  (segment (start 138.8872 134.5184) (end 143.57001 134.5184) (width 1.83) (layer F.Cu) (net 11))
+  (segment (start 156.47321 121.6152) (end 167.999812 121.6152) (width 1.83) (layer F.Cu) (net 11))
+  (segment (start 143.57001 134.5184) (end 156.47321 121.6152) (width 1.83) (layer F.Cu) (net 11))
+  (segment (start 167.999812 121.6152) (end 184.459012 105.156) (width 1.83) (layer F.Cu) (net 11))
+  (segment (start 184.459012 105.156) (end 193.52514 105.156) (width 1.83) (layer F.Cu) (net 11))
+  (segment (start 193.52514 105.156) (end 201.85634 96.8248) (width 1.83) (layer F.Cu) (net 11))
+  (segment (start 136.046329 111.502071) (end 157.199331 90.349069) (width 0.25) (layer F.Cu) (net 17))
+  (segment (start 136.995261 117.852071) (end 136.046329 116.903139) (width 0.25) (layer F.Cu) (net 17))
+  (segment (start 136.995261 135.327271) (end 136.995261 117.852071) (width 0.25) (layer F.Cu) (net 17))
+  (segment (start 158.0388 70.4088) (end 164.56764 70.4088) (width 0.25) (layer F.Cu) (net 17))
+  (segment (start 201.238457 95.584789) (end 202.369969 95.584789) (width 0.25) (layer F.Cu) (net 17))
+  (segment (start 203.096351 97.338429) (end 194.038768 106.39601) (width 0.25) (layer F.Cu) (net 17))
+  (segment (start 138.011261 136.343271) (end 136.995261 135.327271) (width 0.25) (layer F.Cu) (net 17))
+  (segment (start 168.51344 122.85521) (end 156.986838 122.85521) (width 0.25) (layer F.Cu) (net 17))
+  (segment (start 184.97264 106.39601) (end 168.51344 122.85521) (width 0.25) (layer F.Cu) (net 17))
+  (segment (start 143.498777 136.343271) (end 138.011261 136.343271) (width 0.25) (layer F.Cu) (net 17))
+  (segment (start 203.096351 96.311171) (end 203.096351 97.338429) (width 0.25) (layer F.Cu) (net 17))
+  (segment (start 194.038768 106.39601) (end 184.97264 106.39601) (width 0.25) (layer F.Cu) (net 17))
+  (segment (start 202.369969 95.584789) (end 203.096351 96.311171) (width 0.25) (layer F.Cu) (net 17))
+  (segment (start 192.653258 86.99959) (end 201.238457 95.584789) (width 0.25) (layer F.Cu) (net 17))
+  (segment (start 181.15843 86.99959) (end 192.653258 86.99959) (width 0.25) (layer F.Cu) (net 17))
+  (segment (start 164.56764 70.4088) (end 181.15843 86.99959) (width 0.25) (layer F.Cu) (net 17))
+  (segment (start 156.986838 122.85521) (end 143.498777 136.343271) (width 0.25) (layer F.Cu) (net 17))
+  (segment (start 136.046329 116.903139) (end 136.046329 111.502071) (width 0.25) (layer F.Cu) (net 17))
+  (segment (start 157.199331 90.349069) (end 158.6992 88.8492) (width 0.25) (layer F.Cu) (net 17))
 )
