File: Connectivity/RFswitch/rfswitch.sch (KiCad schematic (older format))
At the start: 9 parts

Commit message: initial sch and layout
Parts:
- removed U? (x4): TLP175A, SO-6, symbol TLP175A
- added C1, C2, C3, C4: CP, Capacitors_SMD:c_elec_5x5.3, symbol CP
- added P6: CONN_01X02, Socket_Strips:Socket_Strip_Angled_1x02, symbol CONN_01X02
- added R1, R2, R3, R4: R, Resistors_SMD:R_1206, symbol R
- added R? (x2): R, symbol R
- added RL1, RL2, RL3, RL4: RM50-xx21, Relays_ThroughHole:Relay_SPDT_Schrack-RP-II-1_RM3-5mm, symbol RM50-xx21
- added SW1, SW2, SW3, SW4: SW_PUSH, Buttons_Switches_SMD:SW_SPST_EVQP0, symbol SW_PUSH
- added U1: LT1129CS8, Socket_Strips:Socket_Strip_Angled_1x07, symbol LT1129CS8
- P1, P2, P3, P4, P5: renamed from P?; footprint (none) -> Sockets_BNC:BNC_Socket_TYCO-AMP
Connections:
- net labels added: +12V, GND
- wire segments 7 -> 83

Commit message: trx model sim matlab initial
Parts:
- gave numbers to parts that had none: 2
Changed lines of the file:
@@
 	5100 6100 5100 6200
 $Comp
-L +12V #PWR01
+L +12V #PWR1
 U 1 1 56CF9F9A
 P 3300 5800
-F 0 "#PWR01" H 3300 5650 50  0001 C CNN
+F 0 "#PWR1" H 3300 5650 50  0001 C CNN
 F 1 "+12V" H 3300 5940 50  0000 C CNN
 F 2 "" H 3300 5800 50  0000 C CNN
@@
 $EndComp
 $Comp
-L GND #PWR02
+L GND #PWR3
 U 1 1 56CFA094
 P 6000 6900
-F 0 "#PWR02" H 6000 6650 50  0001 C CNN
+F 0 "#PWR3" H 6000 6650 50  0001 C CNN
 F 1 "GND" H 6000 6750 50  0000 C CNN
 F 2 "" H 6000 6900 50  0000 C CNN
@@
 Connection ~ 4610 2500
 $Comp
-L GND #PWR?
+L GND #PWR2
 U 1 1 56CFCA40
 P 5800 5520
-F 0 "#PWR?" H 5800 5270 50  0001 C CNN
+F 0 "#PWR2" H 5800 5270 50  0001 C CNN
 F 1 "GND" H 5800 5370 50  0000 C CNN
 F 2 "" H 5800 5520 50  0000 C CNN
@@
 	3300 5800 3300 5950
 $Comp
-L R R?
+L R R6
 U 1 1 56CFCE65
 P 4630 5950
-F 0 "R?" V 4710 5950 50  0000 C CNN
+F 0 "R6" V 4710 5950 50  0000 C CNN
 F 1 "R" V 4630 5950 50  0000 C CNN
 F 2 "" V 4560 5950 50  0000 C CNN
@@
 $EndComp
 $Comp
-L R R?
+L R R5
 U 1 1 56CFCEE0
 P 4480 6170
-F 0 "R?" H 4560 6170 50  0000 C CNN
+F 0 "R5" H 4560 6170 50  0000 C CNN
 F 1 "R" V 4480 6170 50  0000 C CNN
 F 2 "" V 4410 6170 50  0000 C CNN
